Commit message: add dynamic controller

File: assets/urdf/106.urdf (robot description, URDF)
Before this commit: robot 106, 14 links, 13 joints
Joints:
- joint 0:virtual::2:seat 1_translation: limit lower=-0.0502704772949219 upper=0.0347295227050781 effort=10 velocity=3 -> lower=-0.0502704772949219 upper=0.0347295227050781 effort=10
- joint 0:virtual::8:gas lift piece 1_rotation: limit lower=-3.141592653589793 upper=3.141592653589793 effort=10 velocity=3 -> lower=-3.141592653589793 upper=3.141592653589793 effort=10
- joint 10:caster 2::5:wheel 3_rotation: limit lower=-3.141592653589793 upper=3.141592653589793 effort=10 velocity=3 -> lower=-3.141592653589793 upper=3.141592653589793 effort=10
- joint 11:caster 3::7:wheel 5_rotation: limit lower=-3.141592653589793 upper=3.141592653589793 effort=10 velocity=3 -> lower=-3.141592653589793 upper=3.141592653589793 effort=10
- joint 12:caster 4::3:wheel 1_rotation: limit lower=-3.141592653589793 upper=3.141592653589793 effort=10 velocity=3 -> lower=-3.141592653589793 upper=3.141592653589793 effort=10
- joint 13:caster 5::6:wheel 4_rotation: limit lower=-3.141592653589793 upper=3.141592653589793 effort=10 velocity=3 -> lower=-3.141592653589793 upper=3.141592653589793 effort=10
- joint 2:seat 1::1:back 1_rotation: limit lower=-0.32986722862692824 upper=0.1413716694115407 effort=10 velocity=3 -> lower=-0.32986722862692824 upper=0.1413716694115407 effort=10
- joint 8:gas lift piece 1::10:caster 2_rotation: limit lower=-3.141592653589793 upper=3.141592653589793 effort=10 velocity=3 -> lower=-3.141592653589793 upper=3.141592653589793 effort=10
- joint 8:gas lift piece 1::11:caster 3_rotation: limit lower=-3.141592653589793 upper=3.141592653589793 effort=10 velocity=3 -> lower=-3.141592653589793 upper=3.141592653589793 effort=10
- joint 8:gas lift piece 1::12:caster 4_rotation: limit lower=-3.141592653589793 upper=3.141592653589793 effort=10 velocity=3 -> lower=-3.141592653589793 upper=3.141592653589793 effort=10
- joint 8:gas lift piece 1::13:caster 5_rotation: limit lower=-3.141592653589793 upper=3.141592653589793 effort=10 velocity=3 -> lower=-3.141592653589793 upper=3.141592653589793 effort=10
- joint 8:gas lift piece 1::9:caster 1_rotation: limit lower=-3.141592653589793 upper=3.141592653589793 effort=10 velocity=3 -> lower=-3.141592653589793 upper=3.141592653589793 effort=10
- joint 9:caster 1::4:wheel 2_rotation: limit lower=-3.141592653589793 upper=3.141592653589793 effort=10 velocity=3 -> lower=-3.141592653589793 upper=3.141592653589793 effort=10

File: assets/urdf/movo_base/movo_base.urdf (robot description, URDF)
Before this commit: robot movo_base, 4 links, 3 joints
Joints:
- joint linear_joint: limit lower=0.0 upper=0.472 effort=1000 velocity=0.20 -> lower=0.0 upper=0.472 effort=1000
