Commit message: add single hand

File: assets/robot/single_hand.urdf (robot description, URDF)
Before this commit: robot movo, 12 links, 10 joints
Links:
- added link root4
- added link root5
- added link root6
Joints:
- added joint p_rotation_joint: type continuous, parent root4, child root5, axis 0 1 0
- added joint r_rotation_joint: type continuous, parent root3, child root4, axis 1 0 0
- added joint right_ee_fixed_joint: type fixed, parent root6, child right_ee_link
- added joint y_rotation_joint: type continuous, parent root5, child root6, axis 0 0 1
- joint x_axis_joint: axis (none) -> 1 0 0; limit (none) -> lower=-10 upper=10 velocity=0.50; origin  -> (none)
- joint y_axis_joint: axis (none) -> 0 1 0; limit (none) -> lower=-10 upper=10 velocity=0.50; origin  -> (none); parent roo1t -> root1
- joint z_axis_joint: axis (none) -> 0 0 1; limit (none) -> lower=-10 upper=10 velocity=0.50; origin  -> (none)
