Commit message: fix xarm and separate controllers and controller parameters

File: assets/robot/xarm6.urdf (robot description, URDF)
Before this commit: robot xarm6_with_gripper, 15 links, 14 joints
Links:
- link xarm_gripper_link_base: geometry collision mesh filename=xarm_gripper/meshes/base_link.STL; visual mesh filename=xarm_gripper/meshes/base_link.STL
