Commit message: add controller fix

File: assets/robot/movo_free_base.urdf (robot description, URDF)
Before this commit: robot movo, 33 links, 32 joints
Joints:
- joint kinect2_ir_joint: origin xyz=0.0245 -0.03325  0.04201 rpy=0 0 0 -> xyz=0.0345 -0.03325  0.05201 rpy=0 0 0
- joint x_axis_joint: limit lower=-10 upper=10 velocity=0.50 -> lower=-10 upper=10 effort=10000 velocity=0.50
- joint y_axis_joint: limit lower=-10 upper=10 velocity=0.50 -> lower=-10 upper=10 effort=10000 velocity=0.50

File: ros_workspace/src/movo_description/urdf/all_robot.urdf (robot description, URDF)
Before this commit: robot movo, 31 links, 30 joints
Links:
- added link root
- added link root1
- added link root2
Joints:
- added joint x_axis_joint: type prismatic, parent root, child root1, axis 1 0 0, limit lower=-10 upper=10 effort=10000 velocity=0.50
- added joint y_axis_joint: type prismatic, parent root1, child root2, axis 0 1 0, limit lower=-10 upper=10 effort=10000 velocity=0.50
- added joint y_rotation_joint: type continuous, parent root2, child base_link, axis 0 0 1
