Commit message: update collision

File: assets/robot/all_robot.urdf (robot description, URDF)
Before this commit: robot movo, 31 links, 30 joints
Links:
- link linear_actuator_link: geometry collision mesh filename=movo_description/meshes/movo_components/collision/movo_uppe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; collision mesh filename=movo_description/meshes/movo_components/collision/movo_uppe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

Commit message: add sapien ros utils

File: assets/robot/all_robot.urdf (robot description, URDF)
Before this commit: robot movo, 31 links, 30 joints
Joints:
- joint linear_joint: limit lower=0.0 upper=0.472 effort=1000 velocity=0.20 -> lower=0.0 upper=0.472 effort=1000
- joint pan_joint: limit lower=-1.570796326794897 upper=1.570796326794897 effort=7.0 velocity=0.907571211 -> lower=-1.570796326794897 upper=1.570796326794897 effort=7.0
- joint right_arm_half_joint: limit lower=-3.14159265 upper=3.14159265 effort=30000.5 velocity=0.691150384 -> lower=-3.14159265 upper=3.14159265 effort=30000.5
- joint right_elbow_joint: limit lower=-2.809 upper=2.809 effort=18000.0 velocity=0.691150384 -> lower=-2.809 upper=2.809 effort=18000.0
- joint right_gripper_finger1_joint: limit lower=0.0 upper=0.986111027 effort=3.0 velocity=1.0 -> lower=0.0 upper=0.986111027 effort=3.0
- joint right_gripper_finger2_joint: limit lower=0.0 upper=0.986111027 effort=3.0 velocity=1.0 -> lower=0.0 upper=0.986111027 effort=3.0
- joint right_gripper_finger3_joint: limit lower=0.0 upper=0.986111027 effort=3.0 velocity=1.0 -> lower=0.0 upper=0.986111027 effort=3.0
- joint right_shoulder_lift_joint: limit lower=-2.238 upper=2.238 effort=30000.5 velocity=0.691150384 -> lower=-2.238 upper=2.238 effort=30000.5
- joint right_shoulder_pan_joint: limit lower=-3.14159265 upper=3.14159265 effort=18000.0 velocity=0.691150384 -> lower=-3.14159265 upper=3.14159265 effort=18000.0
- joint right_wrist_3_joint: limit lower=-3.14159265 upper=3.14159265 effort=60000.8 velocity=0.921533845 -> lower=-3.14159265 upper=3.14159265 effort=60000.8
- joint right_wrist_spherical_1_joint: limit lower=-3.14159265 upper=3.14159265 effort=60000.8 velocity=0.921533845 -> lower=-3.14159265 upper=3.14159265 effort=60000.8
- joint right_wrist_spherical_2_joint: limit lower=-2.78 upper=2.78 effort=60000.8 velocity=0.921533845 -> lower=-2.78 upper=2.78 effort=60000.8
- joint tilt_joint: limit lower=-1.570796326794897 upper=1.570796326794897 effort=7.0 velocity=0.907571211 -> lower=-1.570796326794897 upper=1.570796326794897 effort=7.0

File: assets/robot/arm_without_gazebo.urdf (robot description, URDF)
Before this commit: robot movo, 17 links, 16 joints
Joints:
- joint right_arm_half_joint: limit lower=-3.14159265 upper=3.14159265 effort=30000.5 velocity=0.691150384 -> lower=-3.14159265 upper=3.14159265 effort=30000.5
- joint right_elbow_joint: limit lower=-2.809 upper=2.809 effort=18000.0 velocity=0.691150384 -> lower=-2.809 upper=2.809 effort=18000.0
- joint right_gripper_finger1_joint: limit lower=0.0 upper=0.986111027 effort=3.0 velocity=1.0 -> lower=0.0 upper=0.986111027 effort=3.0
- joint right_gripper_finger2_joint: limit lower=0.0 upper=0.986111027 effort=3.0 velocity=1.0 -> lower=0.0 upper=0.986111027 effort=3.0
- joint right_gripper_finger3_joint: limit lower=0.0 upper=0.986111027 effort=3.0 velocity=1.0 -> lower=0.0 upper=0.986111027 effort=3.0
- joint right_shoulder_lift_joint: limit lower=-2.238 upper=2.238 effort=30000.5 velocity=0.691150384 -> lower=-2.238 upper=2.238 effort=30000.5
- joint right_shoulder_pan_joint: limit lower=-3.14159265 upper=3.14159265 effort=18000.0 velocity=0.691150384 -> lower=-3.14159265 upper=3.14159265 effort=18000.0
- joint right_wrist_3_joint: limit lower=-3.14159265 upper=3.14159265 effort=60000.8 velocity=0.921533845 -> lower=-3.14159265 upper=3.14159265 effort=60000.8
- joint right_wrist_spherical_1_joint: limit lower=-3.14159265 upper=3.14159265 effort=60000.8 velocity=0.921533845 -> lower=-3.14159265 upper=3.14159265 effort=60000.8
- joint right_wrist_spherical_2_joint: limit lower=-2.78 upper=2.78 effort=60000.8 velocity=0.921533845 -> lower=-2.78 upper=2.78 effort=60000.8

File: assets/robot/test.urdf (robot description, URDF)
Before this commit: robot movo, 17 links, 16 joints
Joints:
- joint right_arm_half_joint: limit lower=-3.14159265 upper=3.14159265 effort=30000.5 velocity=0.691150384 -> lower=-3.14159265 upper=3.14159265 effort=30000.5
- joint right_elbow_joint: limit lower=-2.809 upper=2.809 effort=18000.0 velocity=0.691150384 -> lower=-2.809 upper=2.809 effort=18000.0
- joint right_gripper_finger1_joint: limit lower=0.0 upper=0.986111027 effort=3.0 velocity=1.0 -> lower=0.0 upper=0.986111027 effort=3.0
- joint right_gripper_finger2_joint: limit lower=0.0 upper=0.986111027 effort=3.0 velocity=1.0 -> lower=0.0 upper=0.986111027 effort=3.0
- joint right_gripper_finger3_joint: limit lower=0.0 upper=0.986111027 effort=3.0 velocity=1.0 -> lower=0.0 upper=0.986111027 effort=3.0
- joint right_shoulder_lift_joint: limit lower=-2.238 upper=2.238 effort=30000.5 velocity=0.691150384 -> lower=-2.238 upper=2.238 effort=30000.5
- joint right_shoulder_pan_joint: limit lower=-3.14159265 upper=3.14159265 effort=18000.0 velocity=0.691150384 -> lower=-3.14159265 upper=3.14159265 effort=18000.0
- joint right_wrist_3_joint: limit lower=-3.14159265 upper=3.14159265 effort=60000.8 velocity=0.921533845 -> lower=-3.14159265 upper=3.14159265 effort=60000.8
- joint right_wrist_spherical_1_joint: limit lower=-3.14159265 upper=3.14159265 effort=60000.8 velocity=0.921533845 -> lower=-3.14159265 upper=3.14159265 effort=60000.8
- joint right_wrist_spherical_2_joint: limit lower=-2.78 upper=2.78 effort=60000.8 velocity=0.921533845 -> lower=-2.78 upper=2.78 effort=60000.8

Commit message: fix KJoint and add xarm

File: assets/robot/all_robot.urdf (robot description, URDF)
Before this commit: robot movo, 31 links, 30 joints
Joints:
- joint right_arm_half_joint: type revolute -> continuous
- joint right_elbow_joint: type revolute -> continuous
- joint right_shoulder_lift_joint: type revolute -> continuous
- joint right_shoulder_pan_joint: type revolute -> continuous
- joint right_wrist_3_joint: type revolute -> continuous
- joint right_wrist_spherical_1_joint: type revolute -> continuous
- joint right_wrist_spherical_2_joint: type revolute -> continuous

Commit message: minor change for joint pub node

File: assets/robot/all_robot.urdf (robot description, URDF)
Before this commit: robot movo, 31 links, 30 joints
Links:
- removed link front_laser_link
- removed link rear_laser_link
- added link lower_body_link, mass 7.753378; visual mesh filename=movo_description/meshes/movo_body/movo_lower_body.dae
- link base_chassis_link: geometry collision mesh filename=movo_description/meshes/movo_components/collision/vector_ba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
Joints:
- removed joint front_laser_joint
- removed joint rear_laser_joint
- added joint lower_body_joint: type fixed, parent base_chassis_link, child lower_body_link, origin xyz=0 0 0 rpy=0 0 0

Commit message: change aspect

File: assets/robot/all_robot.urdf (robot description, URDF)
Before this commit: robot movo, 30 links, 29 joints
Links:
- link base_chassis_link: geometry collision mesh filename=movo_description/meshes/movo_components/collision/vector_ba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; visual mesh filename=movo_description/meshes/movo_components/visual/vector_base.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

Commit message: add setup python

File: assets/robot/all_robot.urdf (robot description, URDF)
Before this commit: robot movo, 30 links, 29 joints
Links:
- link right_wrist_3_link: geometry 
