Commit message: clean assets folder and move to assets_local. Assets_local is only used for developer

File: assets/robot/locobot_lite_description.urdf (robot description, URDF)
Before this commit: robot locobot_lite, 24 links, 23 joints
Links:
- link ar_tag: geometry collision mesh filename=locobot_description/meshes/ar_tag.STL; visual mesh filename=locobot_description/meshes/ar_tag.STL
- link arm_base_link: geometry collision mesh filename=locobot_description/meshes/arm_base_link.STL; visual mesh filename=locobot_description/meshes/arm_base_link.STL
- link base_link: geometry collision cylinder length=0.0611632 radius=0.16495; visual mesh filename=ca_description/meshes/create_2.dae
- link bottom_plate: geometry collision mesh filename=locobot_description/meshes/base_link.STL; visual mesh filename=locobot_description/meshes/base_link.STL
- link camera_link: geometry collision mesh filename=locobot_description/meshes/camera_link.STL; visual mesh filename=locobot_description/meshes/camera_link.STL
- link elbow_link: geometry collision mesh filename=locobot_description/meshes/elbow_link.STL; visual mesh filename=locobot_description/meshes/elbow_link.STL
- link finger_l: geometry collision mesh filename=locobot_description/meshes/finger_l.STL; visual mesh filename=locobot_description/meshes/finger_l.STL
- link finger_r: geometry collision mesh filename=locobot_description/meshes/finger_r.STL; visual mesh filename=locobot_description/meshes/finger_r.STL
- link forearm_link: geometry collision mesh filename=locobot_description/meshes/forearm_link.STL; visual mesh filename=locobot_description/meshes/forearm_link.STL
- link gripper_link: geometry collision mesh filename=locobot_description/meshes/gripper_link.STL; visual mesh filename=locobot_description/meshes/gripper_link.STL
- link head_pan_link: geometry collision mesh filename=locobot_description/meshes/yaw_link.STL; visual mesh filename=locobot_description/meshes/yaw_link.STL
- link head_tilt_link: geometry collision mesh filename=locobot_description/meshes/roll_link.STL; visual mesh filename=locobot_description/meshes/roll_link.STL
- link shoulder_link: geometry collision mesh filename=locobot_description/meshes/shoulder_link.STL; visual mesh filename=locobot_description/meshes/shoulder_link.STL
- link wrist_link: geometry collision mesh filename=locobot_description/meshes/wrist_link.STL; visual mesh filename=locobot_description/meshes/wrist_link.STL
